File: fightstick_v2.kicad_sch (KiCad schematic)
At the start: 158 parts, among them J1 USB_C_Receptacle_USB2.0, J2 Conn_01x04, J3 Conn_01x03, J9 Conn_01x05, SW1 SW_Push, SW10 SW_Push, SW11 SW_Push, SW12 SW_Push, SW13 SW_Push, SW14 SW_Push, SW15 SW_Push, SW16 SW_Push, SW17 SW_Push, SW19 SW_Push, SW2 SW_Push, SW3 SW_Push, SW4 SW_Push, SW5 SW_Push, SW6 SW_Push, SW7 SW_Push, SW8 SW_Push, SW9 SW_Push, U1 XC6206PxxxMR, U2 W25Q128JVS, U3 RP2040, U4 SRV05-4, U5 74AHCT1G125, Y1 12MHz

Commit message: tried creating a bom
Other:
- moved on the sheet: C17, H1, H10, H2, H3, H4, H5, H6, H7, H8, H9, J2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

Commit message: v0.1, shipping this
Parts:
- C17: footprint Capacitor_SMD:C_0402_1005Metric -> Capacitor_SMD:C_0805_2012Metric; LCSC C15525 -> C15850
Changed lines of the file:
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@@
       (effects (font (size 1.27 1.27)) (justify left))
     )
-    (property "Footprint" "Capacitor_SMD:C_0402_1005Metric" (id 2) (at 127.9652 34.29 0)
+    (property "Footprint" "Capacitor_SMD:C_0805_2012Metric" (id 2) (at 127.9652 34.29 0)
       (effects (font (size 1.27 1.27)) hide)
     )
@@
       (effects (font (size 1.27 1.27)) hide)
     )
-    (property "LCSC" "C15525" (id 4) (at 127 30.48 0)
+    (property "LCSC" "C15850" (id 4) (at 127 30.48 0)
       (effects (font (size 1.27 1.27)) hide)
     )
@@
     )
     (path "/112bc1fe-177e-466c-81c8-a1331d7cc088"
-      (reference "C17") (unit 1) (value "10uF") (footprint "Capacitor_SMD:C_0402_1005Metric")
+      (reference "C17") (unit 1) (value "10uF") (footprint "Capacitor_SMD:C_0805_2012Metric")
     )
     (path "/f7ba96e6-91a2-499a-8627-1f98ce6ee969"

Commit message: replaced leds with sk6812-ec20s
Parts:
- D13, D14, D15, D16, D17, D18, D19, D20, D21, D22, D23, D24, D25, D26, D27, D28, D29, D30, D31, D32, D33, D34, D35, D36, D37, D38, D39, D40, D41, D42, D43, D44, D45, D46, D47, D48, D49, D50, D51, D52: value WS2812C-2020 -> SK6812; footprint components:LED_WS2812-2020 -> LED_SMD:LED_SK6805_PLCC4_2.4x2.7mm_P1.3mm; symbol LED:WS2812B -> LED:SK6812; LCSC C81598 -> C2909058
- U3: LCSC C97521 -> C2040
Connections:
- net +5V: now also D13.3 (VDD), D14.3 (VDD), D15.3 (VDD), D16.3 (VDD), D17.3 (VDD), D18.3 (VDD), D19.3 (VDD), D20.3 (VDD), D21.3 (VDD), D22.3 (VDD), D23.3 (VDD), D24.3 (VDD), D25.3 (VDD), D26.3 (VDD), D27.3 (VDD), D28.3 (VDD), D29.3 (VDD), D30.3 (VDD), D31.3 (VDD), D32.3 (VDD), D33.3 (VDD), D34.3 (VDD), D35.3 (VDD), D36.3 (VDD), D37.3 (VDD), D38.3 (VDD), D39.3 (VDD), D40.3 (VDD), D41.3 (VDD), D42.3 (VDD), D43.3 (VDD), D44.3 (VDD), D45.3 (VDD), D46.3 (VDD), D47.3 (VDD), D48.3 (VDD), D49.3 (VDD), D50.3 (VDD), D51.3 (VDD), D52.3 (VDD); no longer D13.1 (VDD), D14.1 (VDD), D15.1 (VDD), D16.1 (VDD), D17.1 (VDD), D18.1 (VDD), D19.1 (VDD), D20.1 (VDD), D21.1 (VDD), D22.1 (VDD), D23.1 (VDD), D24.1 (VDD), D25.1 (VDD), D26.1 (VDD), D27.1 (VDD), D28.1 (VDD), D29.1 (VDD), D30.1 (VDD), D31.1 (VDD), D32.1 (VDD), D33.1 (VDD), D34.1 (VDD), D35.1 (VDD), D36.1 (VDD), D37.1 (VDD), D38.1 (VDD), D39.1 (VDD), D40.1 (VDD), D41.1 (VDD), D42.1 (VDD), D43.1 (VDD), D44.1 (VDD), D45.1 (VDD), D46.1 (VDD), D47.1 (VDD), D48.1 (VDD), D49.1 (VDD), D50.1 (VDD), D51.1 (VDD), D52.1 (VDD)
- net D_ARGB_5V: now also D13.2 (DIN); no longer D13.4 (DIN)
- net GND: now also D13.1 (VSS), D14.1 (VSS), D15.1 (VSS), D16.1 (VSS), D17.1 (VSS), D18.1 (VSS), D19.1 (VSS), D20.1 (VSS), D21.1 (VSS), D22.1 (VSS), D23.1 (VSS), D24.1 (VSS), D25.1 (VSS), D26.1 (VSS), D27.1 (VSS), D28.1 (VSS), D29.1 (VSS), D30.1 (VSS), D31.1 (VSS), D32.1 (VSS), D33.1 (VSS), D34.1 (VSS), D35.1 (VSS), D36.1 (VSS), D37.1 (VSS), D38.1 (VSS), D39.1 (VSS), D40.1 (VSS), D41.1 (VSS), D42.1 (VSS), D43.1 (VSS), D44.1 (VSS), D45.1 (VSS), D46.1 (VSS), D47.1 (VSS), D48.1 (VSS), D49.1 (VSS), D50.1 (VSS), D51.1 (VSS), D52.1 (VSS); no longer D13.3 (VSS), D14.3 (VSS), D15.3 (VSS), D16.3 (VSS), D17.3 (VSS), D18.3 (VSS), D19.3 (VSS), D20.3 (VSS), D21.3 (VSS), D22.3 (VSS), D23.3 (VSS), D24.3 (VSS), D25.3 (VSS), D26.3 (VSS), D27.3 (VSS), D28.3 (VSS), D29.3 (VSS), D30.3 (VSS), D31.3 (VSS), D32.3 (VSS), D33.3 (VSS), D34.3 (VSS), D35.3 (VSS), D36.3 (VSS), D37.3 (VSS), D38.3 (VSS), D39.3 (VSS), D40.3 (VSS), D41.3 (VSS), D42.3 (VSS), D43.3 (VSS), D44.3 (VSS), D45.3 (VSS), D46.3 (VSS), D47.3 (VSS), D48.3 (VSS), D49.3 (VSS), D50.3 (VSS), D51.3 (VSS), D52.3 (VSS)
- net at D49.2 (DIN): now also D45.4 (DOUT); no longer D14.4 (DIN)
- net at D49.4 (DOUT): now also D14.2 (DIN); no longer D45.2 (DOUT)
- net at D39.2 (DIN): now also D35.4 (DOUT); no longer D43.4 (DIN)
- net at D39.4 (DOUT): now also D43.2 (DIN); no longer D35.2 (DOUT)
- net at D17.4 (DOUT): now also D21.2 (DIN); no longer D13.2 (DOUT)
- net at D36.2 (DIN): now also D32.4 (DOUT); no longer D40.4 (DIN)
- net at D36.4 (DOUT): now also D40.2 (DIN); no longer D32.2 (DOUT)
- net at D18.2 (DIN): now also D14.4 (DOUT); no longer D22.4 (DIN)
- net at D18.4 (DOUT): now also D22.2 (DIN); no longer D14.2 (DOUT)
- net at D25.2 (DIN): now also D21.4 (DOUT); no longer D29.4 (DIN)
- net at D25.4 (DOUT): now also D29.2 (DIN); no longer D21.2 (DOUT)
- net at D41.2 (DIN): now also D37.4 (DOUT); no longer D45.4 (DIN)
- net at D24.2 (DIN): now also D20.4 (DOUT); no longer D28.4 (DIN)
- net at D24.4 (DOUT): now also D28.2 (DIN); no longer D20.2 (DOUT)
- net at D16.2 (DIN): now also D51.4 (DOUT); no longer D20.4 (DIN)
- net at D42.2 (DIN): now also D38.4 (DOUT); no longer D46.4 (DIN)
- net at D42.4 (DOUT): now also D46.2 (DIN); no longer D38.2 (DOUT)
- net at D31.2 (DIN): now also D27.4 (DOUT); no longer D35.4 (DIN)
- net at D31.4 (DOUT): now also D35.2 (DIN); no longer D27.2 (DOUT)
- net at D47.4 (DOUT): now also D51.2 (DIN); no longer D43.2 (DOUT)
- net at D17.2 (DIN): now also D13.4 (DOUT); no longer D21.4 (DIN)
- net at D52.2 (DIN): now also D48.4 (DOUT)
- net at D52.4 (DOUT): no longer D48.2 (DOUT)
- net at D44.2 (DIN): now also D40.4 (DOUT); no longer D48.4 (DIN)
- net at D44.4 (DOUT): now also D48.2 (DIN); no longer D40.2 (DOUT)
- net at D16.4 (DOUT): now also D20.2 (DIN); no longer D51.2 (DOUT)
- net at D26.2 (DIN): now also D22.4 (DOUT); no longer D30.4 (DIN)
- net at D26.4 (DOUT): now also D30.2 (DIN); no longer D22.2 (DOUT)
- net at D15.2 (DIN): now also D50.4 (DOUT); no longer D19.4 (DIN)
- net at D15.4 (DOUT): now also D19.2 (DIN); no longer D50.2 (DOUT)
- net at D47.2 (DIN): now also D43.4 (DOUT); no longer D51.4 (DIN)
- net at D23.4 (DOUT): now also D27.2 (DIN); no longer D19.2 (DOUT)
- net at D41.4 (DOUT): now also D45.2 (DIN); no longer D37.2 (DOUT)
- net at D34.4 (DOUT): now also D38.2 (DIN); no longer D30.2 (DOUT)
- net at D33.2 (DIN): now also D29.4 (DOUT); no longer D37.4 (DIN)
- net at D23.2 (DIN): now also D19.4 (DOUT); no longer D27.4 (DIN)
- net at D34.2 (DIN): now also D30.4 (DOUT); no longer D38.4 (DIN)
- net at D33.4 (DOUT): now also D37.2 (DIN); no longer D29.2 (DOUT)
- new net: D28.4 (DOUT), D32.2 (DIN)
- new net: D46.4 (DOUT), D50.2 (DIN)
